File: hardware/7seg-control/7seg-control.kicad_pcb (KiCad board)
At the start: 2 copper layers, 50.8 x 76.2 mm, 57 parts, among them J101 CH0, J102 I2C THRU, J103 CH1, J104 I2C THRU, J105 CH2, J106 CH3, J107 CH5, J108 Conn_02x04_Odd_Even, J109 CH6, J110 Conn_02x04_Odd_Even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

Commit message: chore: add hardware files and config changes
Parts:
- removed JP102: A2, Connector_PinHeader_2.54mm:PinHeader_1x03_P2.54mm_Vertical
- removed JP103: A1, Connector_PinHeader_2.54mm:PinHeader_1x03_P2.54mm_Vertical
- removed JP104: A0, Connector_PinHeader_2.54mm:PinHeader_1x03_P2.54mm_Vertical
- removed JP105: A0, Connector_PinHeader_2.54mm:PinHeader_1x02_P2.54mm_Vertical
- removed JP106: A1, Connector_PinHeader_2.54mm:PinHeader_1x02_P2.54mm_Vertical
- removed JP107: A2, Connector_PinHeader_2.54mm:PinHeader_1x02_P2.54mm_Vertical
- added J116: Conn_02x03_Odd_Even, Connector_PinHeader_2.54mm:PinHeader_2x03_P2.54mm_Vertical, F.Cu at (127.5, 56.7)
- added J117: Conn_02x03_Odd_Even, Connector_PinHeader_2.54mm:PinHeader_2x03_P2.54mm_Vertical, F.Cu at (120.5, 56.7)
- added JP101: A2, Connector_PinHeader_2.54mm:PinHeader_1x03_P2.54mm_Vertical, F.Cu at (117.9, 56.7)
- turned R125 to -90 degrees
Routing:
- net VCC: track 157.1 -> 167.8 mm
- net COM0: track 44.6 -> 49.6 mm
- net Net-(J117-Pin_5): track 31.1 -> 33.7 mm
- net ROW0: track 57.2 -> 59.6 mm
- net Net-(J117-Pin_1): track 34.0 -> 32.6 mm
- net Net-(J116-Pin_4): track 3.03 -> 4.22 mm
- net Net-(J117-Pin_3): track 35.1 -> 36.2 mm
- net ROW1: track 51.8 -> 52.8 mm
- net GND: track 146.9 -> 145.8 mm, vias 18 -> 17
- net ROW2: track 46.3 -> 47.3 mm
- net Net-(J116-Pin_6): track 3.03 -> 3.97 mm
- net ROW13: track 35.5 -> 36.0 mm
Other:
- board text added: "<<DIGITI 0.4.1>> 2025-10-02 UMEMOTO LLC"
- board text added: "A0 A1 A2"
- board text added: "EXPANDER GND VCC"
- board text removed: "<<DIGITI 0.4.0>> 2025-09-05 UMEMOTO LLC"
- board text removed: "EXPANDER VCC GND"
