File: hardware/7seg-control/7seg-control.kicad_sch (KiCad schematic)
At the start: 57 parts, among them J101 CH0, J102 I2C THRU, J103 CH1, J104 I2C THRU, J105 CH2, J106 CH3, J107 CH5, J108 Conn_02x04_Odd_Even, J109 CH6, J110 Conn_02x04_Odd_Even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

Commit message: chore: add hardware files and config changes
Parts:
- removed JP102: A2, Connector_PinHeader_2.54mm:PinHeader_1x03_P2.54mm_Vertical, symbol Connector:Conn_01x03_Pin
- removed JP103: A1, Connector_PinHeader_2.54mm:PinHeader_1x03_P2.54mm_Vertical, symbol Connector:Conn_01x03_Pin
- removed JP104: A0, Connector_PinHeader_2.54mm:PinHeader_1x03_P2.54mm_Vertical, symbol Connector:Conn_01x03_Pin
- removed JP105: A0, Connector_PinHeader_2.54mm:PinHeader_1x02_P2.54mm_Vertical, symbol Connector:Conn_01x02_Pin
- removed JP106: A1, Connector_PinHeader_2.54mm:PinHeader_1x02_P2.54mm_Vertical, symbol Connector:Conn_01x02_Pin
- removed JP107: A2, Connector_PinHeader_2.54mm:PinHeader_1x02_P2.54mm_Vertical, symbol Connector:Conn_01x02_Pin
- added J116, J117: Conn_02x03_Odd_Even, Connector_PinHeader_2.54mm:PinHeader_2x03_P2.54mm_Vertical, symbol Connector_Generic:Conn_02x03_Odd_Even
- added JP101: A2, Connector_PinHeader_2.54mm:PinHeader_1x03_P2.54mm_Vertical, symbol Connector:Conn_01x03_Pin
Connections:
- net GND: now also JP101.1 (Pin_1), JP101.2 (Pin_2), JP101.3 (Pin_3)
- net ROW0: now also J116.1 (Pin_1)
- net ROW1: now also J116.3 (Pin_3)
- net ROW2: now also J116.5 (Pin_5)
- net VCC: now also J117.2 (Pin_2), J117.4 (Pin_4), J117.6 (Pin_6)
- net at R126.2: now also J116.2 (Pin_2)
- net at R125.2: now also J116.4 (Pin_4)
- net at U102.1 (A0): now also J117.1 (Pin_1)
- net at U102.2 (A1): now also J117.3 (Pin_3)
- net at U102.21 (A2): now also J117.5 (Pin_5)
- net at R124.2: now also J116.6 (Pin_6)
Other:
- note added: "A2 A1 A0"
- moved on the sheet: C105, H101, R125, R126
