File: hardware/7seg-led/7seg-led.kicad_pcb (KiCad board)
At the start: 2 copper layers, 50.8 x 76.2 mm, 15 parts, among them J201 Conn_02x04_Odd_Even, J202 Conn_02x04_Odd_Even, J203 Conn_02x04_Odd_Even, U201 DA56-11EWA, U202 DA56-11EWA, U203 DA56-11EWA, U204 DA56-11EWA, U205 DA56-11EWA, U206 DA56-11EWA, U207 DA56-11EWA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

Commit message: chore: add hardware files and config changes
Routing:
- net COM0: track 283.0 -> 292.5 mm
- net COM4: track 276.9 -> 282.7 mm
- net COM1: track 271.0 -> 276.8 mm
- net COM7: track 287.4 -> 290.9 mm
- net COM5: track 290.5 -> 293.8 mm
- net COM2: track 279.7 -> 282.7 mm
- net COM3: track 288.2 -> 289.9 mm
- net COM6: track 275.6 -> 277.0 mm
Other:
- board text added: "2025.10.02 << DIGITI >> 0.2.2"
- board text removed: "2025.07.11 << DIGITI >> 0.2.1"
