File: hardware/7seg-power/7seg-power.kicad_pcb (KiCad board)
At the start: 2 copper layers, 50.8 x 76.2 mm, 23 parts, among them J101 VBUS, J102 USB_C_Receptacle_PowerOnly_6P, J103 +5V, U101 K7805M-2000, U103 CH221K

Commit message: chore: add hardware files and config changes
Parts:
- removed H101: VBUS, MountingHole:MountingHole_3.2mm_M3_DIN965_Pad
- removed H105: +5V, MountingHole:MountingHole_3.2mm_M3_DIN965_Pad
- added H106: MountingHole, MountingHole:MountingHole_3.2mm_M3, F.Cu at (107.0, 58.9)
- added H107: MountingHole, MountingHole:MountingHole_3.2mm_M3, F.Cu at (144.0, 58.9)
- added J104: VBUS, 7seg-panel:Generic_XH_S2B-XH-A-1_1x02_P2.50mm_Horizontal, F.Cu at (127.2, 65.3)
- C106: footprint Capacitor_SMD:C_Elec_6.3x5.8 -> Capacitor_THT:CP_Radial_D10.0mm_P5.00mm_P7.50mm; moved to F.Cu
- J102: footprint Connector_USB:USB_C_Receptacle_GCT_USB4125-xx-x-0190_6P_TopMnt_Horizontal -> Connector_USB:USB_C_Receptacle_HRO_TYPE-C-31-M-17
- moved C101 13.5 mm to (117.8, 92.7)
- moved C105 13.5 mm to (111.9, 92.7)
- moved C106 12.6 mm to (112.1, 85.3)
- moved R108 12.3 mm to (134.1, 71.4), turned to 90 degrees
- moved C104 12.2 mm to (112.4, 95.4)
- moved C103 12.1 mm to (116.8, 95.3)
- moved U101 11.8 mm to (117.4, 98.8)
- moved J103 1.58 mm to (118.5, 65.3)
Routing:
- net Net-(U103-VDD): track 30.2 -> 17.4 mm
- net GND: track 138.9 -> 140.6 mm, vias 3 -> 18
- net Net-(J102-CC2): track 36.7 -> 37.3 mm
Other:
- board text added: "<<DIGITI POWER 0.4.2 >> 2025-10-02 UMEMOTO LLC"
- board text removed: "<<DIGITI POWER 0.4.1 >> 2025-09-05 UMEMOTO LLC"
