File: hardware/7seg-power/7seg-power.kicad_sch (KiCad schematic)
At the start: 23 parts, among them J101 VBUS, J102 USB_C_Receptacle_PowerOnly_6P, J103 +5V, U101 K7805M-2000, U103 CH221K

Commit message: chore: add hardware files and config changes
Parts:
- removed H101: VBUS, MountingHole:MountingHole_3.2mm_M3_DIN965_Pad, symbol Mechanical:MountingHole_Pad_MP
- removed H105: +5V, MountingHole:MountingHole_3.2mm_M3_DIN965_Pad, symbol Mechanical:MountingHole_Pad_MP
- added H106, H107: MountingHole, MountingHole:MountingHole_3.2mm_M3, symbol Mechanical:MountingHole
- added J104: VBUS, 7seg-panel:Generic_XH_S2B-XH-A-1_1x02_P2.50mm_Horizontal, symbol Connector_Generic:Conn_01x02
- C106: footprint Capacitor_SMD:C_Elec_6.3x5.8 -> Capacitor_THT:CP_Radial_D10.0mm_P5.00mm_P7.50mm
- J102: footprint Connector_USB:USB_C_Receptacle_GCT_USB4125-xx-x-0190_6P_TopMnt_Horizontal -> Connector_USB:USB_C_Receptacle_HRO_TYPE-C-31-M-17
Connections:
- net GND: now also J104.1 (Pin_1)
- net VBUS: now also J104.2 (Pin_2)
Other:
- moved on the sheet: H102
