File: hardware/7seg-panel-control-040-dual/7seg-panel-control-040-dual.kicad_sch (KiCad schematic)
At the start: 44 parts, among them J102 I2C, J103 I2C, J104 I2C, J105 I2C, J108 Conn_02x04_Odd_Even, J109 Conn_02x04_Odd_Even, J110 Conn_02x04_Odd_Even, J111 Conn_02x04_Odd_Even, J112 Conn_02x04_Odd_Even, J113 Conn_02x04_Odd_Even, J114 +5V, J115 +5V, J116 Conn_02x03_Odd_Even, J117 +5V, J118 I2C, J119 +5V, J120 I2C, J121 I2C, J122 I2C, J123 Conn_02x03_Odd_Even, U103 HT16K33-28-SOPA, U104 HT16K33-28-SOPA

Commit message: added pcb designs
Parts:
- removed J102, J103, J104, J105, J118, J120: I2C, Connector_JST:JST_XH_B2B-XH-AM_1x02_P2.50mm_Vertical, symbol Connector_Generic:Conn_01x02
- removed J114, J115: +5V, Connector_JST:JST_XH_B2B-XH-AM_1x02_P2.50mm_Vertical, symbol Connector_Generic:Conn_01x02
- J107: renamed from J121; footprint Connector_JST:JST_XH_B2B-XH-AM_1x02_P2.50mm_Vertical -> 7seg-panel:Generic_XH_S2B-XH-A-1_1x02_P2.50mm_Horizontal
- J113: renamed from J117; footprint Connector_JST:JST_XH_B2B-XH-AM_1x02_P2.50mm_Vertical -> 7seg-panel:Generic_XH_S2B-XH-A-1_1x02_P2.50mm_Horizontal
- J114: renamed from J119; footprint Connector_JST:JST_XH_B2B-XH-AM_1x02_P2.50mm_Vertical -> 7seg-panel:Generic_XH_S2B-XH-A-1_1x02_P2.50mm_Horizontal
- J117: renamed from J122; footprint Connector_JST:JST_XH_B2B-XH-AM_1x02_P2.50mm_Vertical -> 7seg-panel:Generic_XH_S2B-XH-A-1_1x02_P2.50mm_Horizontal
- renumbered C103 to C102, C104 to C103, C106 to C104, C107 to C106, C108 to C107, J108 to J102, J110 to J105, J112 to J108, J116 to J110, J109 to J112, J111 to J115, J113 to J118, J123 to J120, R124 to R102, R125 to R103, R126 to R104, R127 to R105, R128 to R106, R129 to R107, U103 to U102, U104 to U103
Connections:
- net COM0: no longer D102.2 (A), J102.1 (Pin_1), U102.2 (COM0/AD)
- net COM1: no longer J102.2 (Pin_2), U102.3 (COM1/KS0)
- net COM2: no longer J102.3 (Pin_3), U102.4 (COM2/KS1)
- net COM3: no longer J102.4 (Pin_4), U102.5 (COM3/KS2)
- net COM4: no longer J102.5 (Pin_5), U102.6 (COM4)
- net COM5: no longer J102.6 (Pin_6), U102.7 (COM5)
- net COM6: no longer J102.7 (Pin_7), U102.8 (COM6)
- net COM7: no longer J102.8 (Pin_8), U102.9 (COM7)
- net ROW0: no longer J105.1 (Pin_1), J110.1 (Pin_1), U102.25 (ROW0/A2)
- net ROW1: no longer J105.2 (Pin_2), J110.3 (Pin_3), U102.24 (ROW1/A1)
- net ROW10: no longer J108.3 (Pin_3), U102.15 (ROW10/K8)
- net ROW11: no longer J108.4 (Pin_4), U102.14 (ROW11/K9)
- net ROW12: no longer J108.5 (Pin_5), U102.13 (ROW12/K10)
- net ROW13: no longer J108.6 (Pin_6), U102.12 (ROW13/K12)
- net ROW14: no longer J108.7 (Pin_7), U102.11 (ROW14/K12)
- net ROW15: no longer J108.8 (Pin_8), U102.10 (ROW15/K13/INT)
- net ROW2: no longer J105.3 (Pin_3), J110.5 (Pin_5), U102.23 (ROW2/A0)
- net ROW3: no longer J105.4 (Pin_4), U102.22 (ROW3/K1)
- net ROW4: no longer J105.5 (Pin_5), U102.21 (ROW4/K2)
- net ROW5: no longer J105.6 (Pin_6), U102.20 (ROW5/K3)
- net ROW6: no longer J105.7 (Pin_7), U102.19 (ROW6/K4)
- net ROW7: no longer J105.8 (Pin_8), U102.18 (ROW7/K5)
- net ROW8: no longer J108.1 (Pin_1), U102.17 (ROW8/K6)
- net ROW9: no longer J108.2 (Pin_2), U102.16 (ROW9/K7)
- new net A_COM0: D102.2 (A), J102.1 (Pin_1), U102.2 (COM0/AD)
- new net A_COM1: J102.2 (Pin_2), U102.3 (COM1/KS0)
- new net A_COM2: J102.3 (Pin_3), U102.4 (COM2/KS1)
- new net A_COM3: J102.4 (Pin_4), U102.5 (COM3/KS2)
- new net A_COM4: J102.5 (Pin_5), U102.6 (COM4)
- new net A_COM5: J102.6 (Pin_6), U102.7 (COM5)
- new net A_COM6: J102.7 (Pin_7), U102.8 (COM6)
- new net A_COM7: J102.8 (Pin_8), U102.9 (COM7)
- new net A_ROW0: J105.1 (Pin_1), J110.1 (Pin_1), U102.25 (ROW0/A2)
- new net A_ROW1: J105.2 (Pin_2), J110.3 (Pin_3), U102.24 (ROW1/A1)
- new net A_ROW10: J108.3 (Pin_3), U102.15 (ROW10/K8)
- new net A_ROW11: J108.4 (Pin_4), U102.14 (ROW11/K9)
- new net A_ROW12: J108.5 (Pin_5), U102.13 (ROW12/K10)
- new net A_ROW13: J108.6 (Pin_6), U102.12 (ROW13/K12)
- new net A_ROW14: J108.7 (Pin_7), U102.11 (ROW14/K12)
- new net A_ROW15: J108.8 (Pin_8), U102.10 (ROW15/K13/INT)
- new net A_ROW2: J105.3 (Pin_3), J110.5 (Pin_5), U102.23 (ROW2/A0)
- new net A_ROW3: J105.4 (Pin_4), U102.22 (ROW3/K1)
- new net A_ROW4: J105.5 (Pin_5), U102.21 (ROW4/K2)
- new net A_ROW5: J105.6 (Pin_6), U102.20 (ROW5/K3)
- new net A_ROW6: J105.7 (Pin_7), U102.19 (ROW6/K4)
- new net A_ROW7: J105.8 (Pin_8), U102.18 (ROW7/K5)
- new net A_ROW8: J108.1 (Pin_1), U102.17 (ROW8/K6)
- new net A_ROW9: J108.2 (Pin_2), U102.16 (ROW9/K7)
Other:
- note removed: "Voltage drops may cause malfunction. Make sure if sufficient power supply capacity. I2C address 0x70 is robust against voltage fluctuations."
